Commit message: Edit files to work

File: src/panda_training/include/extra.xacro (robot description, xacro)
@@ -2,5 +2,4 @@
 <robot xmlns:xacro="http://www.ros.org/wiki/xacro" name="panda">
     <xacro:arg name="initial_positions_file" default="initial_positions.yaml" />
-    <xacro:arg name="ros2_control_hardware_type" default="mock_components" />
     <!-- Import panda urdf file -->
     <xacro:include filename="$(find moveit_resources_panda_description)/urdf/panda.urdf" />
@@ -9,8 +8,6 @@
     <!-- overhead position -->
     <!-- <xacro:kinect_camera parent_link="panda_link0" cam_px="0.5" cam_pz="0.7" cam_op="4.71219632679"/> -->
-    <!-- Import panda ros2_control description -->
+    <!-- Import control_xacro -->
     <xacro:include filename="panda.ros2_control.xacro" />
-    <xacro:include filename="panda_hand.ros2_control.xacro" />
-    <xacro:panda_ros2_control name="PandaFakeSystem" initial_positions_file="$(arg initial_positions_file)" ros2_control_hardware_type="$(arg ros2_control_hardware_type)"/>
-    <xacro:panda_hand_ros2_control name="PandaHandFakeSystem" ros2_control_hardware_type="$(arg ros2_control_hardware_type)"/>
+    <xacro:panda_ros2_control name="FakeSystem" initial_positions_file="$(arg initial_positions_file)"/>
 </robot>

File: src/robot_moveit_config/config/lab.urdf.xacro (robot description, xacro)
@@ -6,5 +6,5 @@
   <xacro:include filename="$(find ur_description)/urdf/ur_macro.xacro"/>
   <!-- import table macro -->
-  <xacro:include filename="$(find lab_description)/urdf/table_macro.xacro"/>
+  <xacro:include filename="$(find launch_robot)/urdf/table_macro.xacro"/>
   <!-- possible 'ur_type' values: ur3, ur3e, ur5, ur5e, ur10, ur10e, ur16e, ur20 -->
   <!-- the default value should raise an error in case this was called without defining the type -->

File: src/robot_moveit_config/config/table_macro.xacro (robot description, xacro)
@@ -11,5 +11,5 @@
         <origin xyz="0.3385 0 0" rpy="0 0 0"/>
         <geometry>
-          <mesh filename="file://$(find lab_description)/meshes/table/table_demo.stl" scale="0.001 0.001 0.001"/>
+          <mesh filename="file://$(find launch_robot)/meshes/table/table_demo.stl" scale="0.001 0.001 0.001"/>
         </geometry>
         <material name="silver">
@@ -20,5 +20,5 @@
         <origin xyz="0.3385 0 0" rpy="0 0 0"/>
         <geometry>
-          <mesh filename="file://$(find lab_description)/meshes/table/table_demo.stl" scale="0.001 0.001 0.001"/>
+          <mesh filename="file://$(find launch_robot)/meshes/table/table_demo.stl" scale="0.001 0.001 0.001"/>
         </geometry>
       </collision>
